File: trim_circuit.kicad_sch (KiCad schematic)
At the start: 10 parts

Commit message: Proof reading and snagging updates
Parts:
- added FB1/1: Fuse, symbol Device:Fuse
- CB?: value CircuitBreaker_1P -> Trim CB; Rating (none) -> 1 Amp
- J?: value PL? -> PL5-B
- J?: value PL? -> PL5-A
- J?: value PL? -> PL4-A
- J?: value PL? -> PL4-B
Connections:
- net Battery +12v: now also FB1/1.1; no longer J?.1 (Pin_1)
- net Ground - TB6/9: now reaches J?.2 (Pin_2)
- net 0v: no longer names the net of CB?.1, J?.1 (Pin_1)
- new net +12v: FB1/1.2, J?.1 (Pin_1)
